Commit message: adjust URDF and separate single/multi AMR parameter file

File: ws/src/pibot_nav/urdf/sim_bot.urdf (robot description, URDF)
Before this commit: robot bot, 7 links, 6 joints
Links:
- link caster_link: mass 0.2 -> 0.13
Joints:
- joint caster_joint: origin xyz=-0.075 0 -0.06 -> xyz=-0.08 0 -0.06
- joint lf_wheel_joint: origin xyz=0.09 0.15 -0.06 -> xyz=0.08 0.15 -0.06
- joint rf_wheel_joint: origin xyz=0.09 -0.15 -0.06 -> xyz=0.08 -0.15 -0.06

Commit message: fix: URDF does not match footprint of params

File: ws/src/pibot_nav/urdf/sim_bot.urdf (robot description, URDF)
Before this commit: robot bot, 7 links, 6 joints
Joints:
- joint laser_joint: origin xyz=0.09 0 0.1 -> xyz=0.08 0 0.1
