Commit message: fix: modify UI configurations for depth camera
- navigator_client.py
  - fix _finishTask not called by using action client in the same callback group
  - fix _sendCancelRequest blocking

- simple_ui/*
  - resize camera image from 160x120 to 640x480
  - adjust topic name not to be global
  - adjust qos of topic "path" as behavior tree changed and planner server publishes only when replanning

- sim_bot.urdf
  - resize camera image from 160x120 to 640x480

- test_low_obstacles.sdf
  - adjust the position of the obstacle for not occupying navigation destinations

- single_nav_w_dcam.launch.py & bot_w_dcam.urdf
  - adjust the topic name of color image to "image_raw" for being compatible with AMR without depth camera
  - increase the height of the depth camera from 0.4m to 0.5m for less blind areas

The service "rtabmap/reset"(type: std_srvs/srv/Empty) can help reduce the impact of point cloud noise. However, using it at the wrong time might cause collision, so it has not been used yet.

File: ws/src/pibot_nav/urdf/bot_w_dcam.urdf (robot description, URDF)
Before this commit: robot bot, 8 links, 7 joints
Joints:
- joint camera_joint: origin xyz=-0.03 0 0.32 rpy=0 0.5236 0 -> xyz=-0.03 0 0.42 rpy=0 0.5236 0

Commit message: feat: change point cloud map construction method from rtabmap to octomap
RTAB-Map is an implementation of SLAM and is conflict with amcl. As Octomap only constructs map, it fits better in the project.

- bot_w_dcam.urdf
  - remove the TF shift for camera_link -> depth_optical_frame(0.08 on z-axis, which is same as base_footprint -> base_link) since octomap does not require it

- octomap_reset.py
  - clear point cloud map if re-localization occurs

- single_nav_w_dcam.launch.py
  - add octomap_server and octomap_reset

File: ws/src/pibot_nav/urdf/bot_w_dcam.urdf (robot description, URDF)
Before this commit: robot bot, 8 links, 7 joints
Joints:
- joint depth_joint: origin xyz=0 0 0.08 rpy=-1.57 0 -1.57 -> xyz=0 0 0 rpy=-1.57 0 -1.57
